Commit message: add baxter render and display

File: data/urdf/baxter.urdf (robot description, URDF)
Before this commit: robot baxter, 58 links, 57 joints
Links:
- removed link world
- link l_gripper_l_finger: geometry collision box size=0.01 0.0135 0.075; collision box size=0.01 0.05 0.017
- link l_gripper_r_finger: geometry collision box size=0.01 0.0135 0.075; collision box size=0.01 0.05 0.017
- link r_gripper_l_finger_tip: geometry collision box size=0.042 0.0065 0.037; visual mesh filename=package://rethink_ee_description/meshes/electric_gripper/fi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
- link r_gripper_r_finger_tip: geometry collision box size=0.042 0.0065 0.037; visual mesh filename=package://rethink_ee_description/meshes/electric_gripper/fi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
Joints:
- removed joint fixed
- joint l_gripper_l_finger_joint: origin xyz=0.0 -0.0014999999999999996 0.02 rpy=0 0 0 -> xyz=0.0 -0.0015 0.02 rpy=0 0 0
- joint l_gripper_l_finger_tip_joint: origin xyz=0.0 0.01725 0.1127 rpy=0 0 0 -> xyz=0.0 0.01725 0.075 rpy=0 0 0
- joint l_gripper_r_finger_joint: origin xyz=0.0 0.0014999999999999996 0.02 rpy=0 0 0 -> xyz=0.0 0.0015 0.02 rpy=0 0 0
- joint l_gripper_r_finger_tip_joint: origin xyz=0.0 -0.01725 0.1127 rpy=0 0 0 -> xyz=0.0 -0.01725 0.075 rpy=0 0 0
- joint left_endpoint: origin xyz=0 0 0.13269999999999998 rpy=0 0 0 -> xyz=0 0 0.095 rpy=0 0 0
- joint r_gripper_l_finger_joint: origin xyz=0.0 -0.011 0.02 rpy=0 0 0 -> xyz=0.0 -0.0015 0.02 rpy=0 0 0
- joint r_gripper_r_finger_joint: origin xyz=0.0 0.011 0.02 rpy=0 0 0 -> xyz=0.0 0.0015 0.02 rpy=0 0 0
