Commit message: fix robot urdf for jsk pr1040

File: data/urdf/pr2.urdf (robot description, URDF)
Before this commit: robot pr2, 88 links, 87 joints
Links:
- removed link projector_wg6802418_child_frame
- removed link projector_wg6802418_frame
- added link head_chain_cb_link
- added link head_mount_kinect_ir_link, mass 0.1; collision sphere radius=0.0005; visual sphere radius=0.0005
- added link head_mount_kinect_ir_optical_frame
- added link head_mount_kinect_rgb_link, mass 0.1; collision sphere radius=0.0005; visual sphere radius=0.0005
- added link head_mount_kinect_rgb_optical_frame
- added link head_mount_link, mass 0.1; collision sphere radius=0.0005; visual mesh filename=package://pr2_description/meshes/sensors/kinect_prosilica_v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 scale=0.001 0.001 0.001
- added link head_mount_prosilica_link, mass 0.1; collision sphere radius=0.0005; visual sphere radius=0.0005
- added link head_mount_prosilica_optical_frame
- added link left_arm_chain_cb_link
- added link right_arm_chain_cb_link
Joints:
- removed joint projector_wg6802418_child_frame_joint
- removed joint projector_wg6802418_frame_joint
- added joint head_chain_cb: type fixed, parent head_tilt_link, child head_chain_cb_link, origin xyz=0.0 0.0 0.0 rpy=0.0 0.0 0.0
- added joint head_mount_joint: type fixed, parent head_plate_frame, child head_mount_link, origin xyz=-0.138 0.0 0.091 rpy=0.0 0.0 0.0
- added joint head_mount_kinect_ir_joint: type fixed, parent head_mount_link, child head_mount_kinect_ir_link, origin xyz=-0.032267 0.0125 0.136453 rpy=0.0 0.0 0.0
- added joint head_mount_kinect_ir_optical_frame_joint: type fixed, parent head_mount_kinect_ir_link, child head_mount_kinect_ir_optical_frame, origin xyz=0.0 0.01 0.0 rpy=-1.57079632679 0.0 -1.57079632679
- added joint head_mount_kinect_rgb_joint: type fixed, parent head_mount_kinect_ir_link, child head_mount_kinect_rgb_link, origin xyz=   -0.00696920244115 -0.0325191168453 -0.0116889085003 rpy=0.0180369961393 -0.029141984173 0.0309389769244
- added joint head_mount_kinect_rgb_optical_frame_joint: type fixed, parent head_mount_kinect_rgb_link, child head_mount_kinect_rgb_optical_frame, origin xyz=0.0 0.0 0.0 rpy=-1.57079632679 0.0 -1.57079632679
- added joint head_mount_prosilica_joint: type fixed, parent head_mount_link, child head_mount_prosilica_link, origin xyz=-0.046457 0.0125 0.088921 rpy=0.0 0.0 0.0
- added joint head_mount_prosilica_optical_frame_joint: type fixed, parent head_mount_prosilica_link, child head_mount_prosilica_optical_frame, origin xyz=0.0 0.0 0.0 rpy=-1.57079632679 0.0 -1.57079632679
- added joint left_arm_chain_cb: type fixed, parent l_wrist_roll_link, child left_arm_chain_cb_link, origin xyz=0.0 0.0 0.0 rpy=0.0 0.0 0.0
- added joint right_arm_chain_cb: type fixed, parent r_wrist_roll_link, child right_arm_chain_cb_link, origin xyz=0.0 0.0 0.0 rpy=0.0 0.0 0.0
